File: PD Board.kicad_pcb (KiCad board)
At the start: 2 copper layers, 69.1 x 47.5 mm, 62 parts, among them J1 XT60-M, J2 XT60-M, J3 XT60-M, J4 XT60-M, J5 XT60-M, J6 XT60-M, P1 B2B-PH-K, P10 B2B-PH-K, P11 B2B-PH-K, P12 B2B-PH-K, P13 B2B-PH-K, P14 B2B-PH-K, P15 B2B-PH-K, P16 B2B-PH-K, P17 B2B-PH-K, P18 B2B-PH-K, P19 B2B-PH-K, P2 B2B-PH-K, P20 B2B-PH-K, P3 B2B-PH-K, P4 B2B-PH-K, P5 B2B-PH-K, P6 B2B-PH-K, P7 B2B-PH-K, P8 B2B-PH-K, P9 B2B-PH-K, U1 MC34063AD, U2 MT3608, U3 MC34063AD, U4 AMS1117-5.0, U5 AMS1117-3.3, U6 AMS1117

Commit message: Uploading V02
Parts:
- removed J6: XT60-M, XT60-M:AMASS_XT60-M
- added J7: XT60PW-M, XT60PW-M:AMASS_XT60PW-M, F.Cu at (110.9, 76.0)
- added P21: B2B-PH-K, B2B-PH-K:B2B-PH-K, F.Cu at (134.1, 125.4)
- added P22: B2B-PH-K, B2B-PH-K:B2B-PH-K, F.Cu at (128.8, 125.4)
- added P23: B2B-PH-K, B2B-PH-K:B2B-PH-K, F.Cu at (123.5, 125.4)
- added P24: B2B-PH-K, B2B-PH-K:B2B-PH-K, F.Cu at (139.3, 125.4)
- added P25: B2B-PH-K, B2B-PH-K:B2B-PH-K, F.Cu at (163.2, 125.4)
- added P26: B2B-PH-K, B2B-PH-K:B2B-PH-K, F.Cu at (157.9, 125.4)
- added P27: B2B-PH-K, B2B-PH-K:B2B-PH-K, F.Cu at (152.5, 125.4)
- added P28: B2B-PH-K, B2B-PH-K:B2B-PH-K, F.Cu at (147.2, 125.4)
- J1, J2, J3, J4, J5: value XT60-M -> XT60PW-M; footprint XT60-M:AMASS_XT60-M -> XT60PW-M:AMASS_XT60PW-M
- moved P20 109.6 mm to (147.2, 132.1), turned to -90 degrees
- moved P19 103.8 mm to (152.5, 132.1), turned to -90 degrees
- moved J5 99.6 mm to (110.9, 93.0), turned to 90 degrees
- moved C10 99.1 mm to (154.8, 118.7)
- moved C9 99.1 mm to (143.9, 114.3)
- moved U4 99.1 mm to (149.3, 116.9)
- moved P18 98.2 mm to (157.9, 132.1), turned to -90 degrees
- moved P1 95.6 mm to (162.4, 87.9)
- moved P17 92.9 mm to (163.2, 132.1), turned to -90 degrees
- moved C5 92.3 mm to (143.6, 91.8)
- moved C3 91.8 mm to (144.7, 101.5)
- moved J4 91.8 mm to (110.9, 110.1), turned to 90 degrees
- moved P4 91.8 mm to (169.3, 82.5)
- moved R4 91.8 mm to (142.2, 95.2)
- moved R3 91.8 mm to (142.2, 98.7)
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Routing:
- net +12V: track 163.8 -> 237.6 mm
- net /9V: track 54.8 -> 17.0 mm
- net /7V: track 48.8 -> 13.8 mm
- net /3.3V: track 24.7 -> 2.62 mm
- net /5V: track 22.3 -> 2.94 mm, vias 0 -> 1
- net /3.7V: track 38.6 -> 19.3 mm
- net GND: track 62.8 -> 58.0 mm, vias 23 -> 135
- net /24V: track 40.6 -> 36.5 mm
- net Net-(U1-DC): track 10.7 -> 8.46 mm
- net Net-(R2-Pad2): track 3.33 -> 4.22 mm
- net Net-(U1-TC): track 2.28 -> 2.82 mm
- added copper zone on F.Cu, net /24V
- added copper zone on F.Cu, net /7V
- added copper zone on F.Cu, net /9V
Other:
- board size 69.1 x 47.5 mm -> 79.1 x 69.6 mm
