File: PD Board.kicad_sch (KiCad schematic)
At the start: 62 parts, among them J1 XT60-M, J2 XT60-M, J3 XT60-M, J4 XT60-M, J5 XT60-M, J6 XT60-M, P1 B2B-PH-K, P10 B2B-PH-K, P11 B2B-PH-K, P12 B2B-PH-K, P13 B2B-PH-K, P14 B2B-PH-K, P15 B2B-PH-K, P16 B2B-PH-K, P17 B2B-PH-K, P18 B2B-PH-K, P19 B2B-PH-K, P2 B2B-PH-K, P20 B2B-PH-K, P3 B2B-PH-K, P4 B2B-PH-K, P5 B2B-PH-K, P6 B2B-PH-K, P7 B2B-PH-K, P8 B2B-PH-K, P9 B2B-PH-K, U1 MC34063AD, U2 MT3608, U3 MC34063AD, U4 AMS1117-5.0, U5 AMS1117-3.3, U6 AMS1117

Commit message: Uploading V02
Parts:
- removed J1, J2, J3, J4, J5, J6: XT60-M, XT60-M:AMASS_XT60-M, symbol XT60-M:XT60-M
- added J1, J2, J3, J4, J5, J7: XT60PW-M, XT60PW-M:AMASS_XT60PW-M, symbol XT60PW-M:XT60PW-M
- added P21, P22, P23, P24, P25, P26, P27, P28: B2B-PH-K, B2B-PH-K:B2B-PH-K, symbol B2B-PH-K:B2B-PH-K
Connections:
- net +12V: now also J1.1 (+), J4.1 (+), J5.1 (+), J7.1 (+)
- net 24V: now also J2.1 (+), J3.1 (+)
- net 3.3V: now also P21.1, P22.1, P23.1, P24.1
- net 5V: now also P25.1, P26.1, P27.1, P28.1
- net GND: now also J1.2 (-), J2.2 (-), J3.2 (-), J4.2 (-), J5.2 (-), J7.2 (-), P21.2, P22.2, P23.2, P24.2, P25.2, P26.2, P27.2, P28.2
Other:
- note added: "Extra Connectors"
- moved on the sheet: C11, C12, C13, C14, R8, R9, U5, U6
